File: vanish.kicad_pcb (KiCad board)
At the start: 2 copper layers, 243.4 x 76.2 mm, 111 parts, among them J1 USB_C_Receptacle_USB2.0, U1 ATmega32U4-AU, Y1 16MHz

Commit message: pcb woirk
Parts:
- removed D40, D42: D_Small, Diode_SMD:D_SOD-123
- removed MX40, MX41, MX43: MX-NoLED, MX_Alps_Hybrid:MX-2U-ReversedStabilizers-NoLED
- removed MX45: MX-NoLED, MX_Alps_Hybrid:MX-1.25U-NoLED
- added C8: 0.1uF, Capacitor_SMD:C_0805_2012Metric, B.Cu at (154.0, 100.3)
- added Ref**: Val**, kbd:M2_HOLE_v3, F.Cu at (93.4, 82.0)
- added Ref**: Val**, kbd:M2_HOLE_v3, F.Cu at (199.0, 82.2)
- added Ref**: Val**, kbd:M2_HOLE_v3, F.Cu at (154.7, 54.8)
- added Ref**: Val**, kbd:M2_HOLE_v3, F.Cu at (124.2, 35.7)
- added Ref**: Val**, kbd:M2_HOLE_v3, F.Cu at (46.5, 70.5)
- added Ref**: Val**, kbd:M2_HOLE_v3, F.Cu at (48.0, 35.7)
- added SW1: SW_Push, rainstuff:tht-reset, F.Cu at (181.7, 102.4)
- MX44: footprint MX_Alps_Hybrid:MX-1U-NoLED -> MX_Alps_Hybrid:MX-1.25U-NoLED
- MX47: footprint MX_Alps_Hybrid:MX-1.25U-NoLED -> MX_Alps_Hybrid:MX-1U-NoLED
- R1: moved to F.Cu
- moved C7 114.7 mm to (148.4, 102.7)
- moved C5 112.6 mm to (148.4, 98.7), turned to 90 degrees
- moved C1 108.8 mm to (152.9, 91.1), turned to 180 degrees
- moved Y1 106.4 mm to (152.9, 87.9), turned to 90 degrees
- moved C2 104.0 mm to (152.9, 84.8), turned to 0 degrees
- moved C4 98.7 mm to (151.6, 102.7), turned to 90 degrees
- moved R1 96.4 mm to (179.7, 105.9), turned to 0 degrees
- moved C6 93.5 mm to (151.6, 98.7)
- moved R4 91.7 mm to (163.7, 103.3), turned to 90 degrees
- moved C3 87.2 mm to (164.0, 98.9), turned to 270 degrees
- moved U1 83.9 mm to (164.3, 83.3), turned to 135 degrees
- moved D11 15.9 mm to (208.8, 28.6)
- moved D41 15.9 mm to (130.2, 85.7)
- moved R5 10.0 mm to (232.3, 25.4), turned to 270 degrees
- moved R6 9.85 mm to (226.0, 25.4), turned to 270 degrees
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Routing:
- net A: track 0.00 -> 226.7 mm
- net D: track 0.00 -> 226.3 mm
- net C: track 0.00 -> 216.8 mm
- net B: track 0.00 -> 216.7 mm
- net VCC: track 76.0 -> 0.00 mm, vias 5 -> 0
- net 10: track 0.00 -> 73.3 mm
- net 1: track 0.00 -> 68.9 mm
- net 2: track 0.00 -> 65.0 mm
- net 5: track 0.00 -> 64.1 mm
- net 9: track 0.00 -> 62.1 mm
- net 0: track 0.00 -> 60.2 mm
- net 3: track 0.00 -> 44.1 mm
- net 7: track 0.00 -> 44.0 mm
- net 4: track 0.00 -> 44.0 mm
- net 8: track 0.00 -> 44.0 mm
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
Commit message: done
Parts:
- removed C2: 22pF, Capacitor_SMD:C_0805_2012Metric
- removed J1: USB_C_Receptacle_USB2.0, Connector_USB:USB_C_Receptacle_GCT_USB4085
- removed Ref** (x7): Val**, kbd:M2_HOLE_v3
- added H1: Hole, kbd:M2_HOLE_v3, F.Cu at (48.0, 35.7)
- added H2: Hole, kbd:M2_HOLE_v3, F.Cu at (46.5, 70.5)
- added H3: Hole, kbd:M2_HOLE_v3, F.Cu at (93.4, 82.0)
- added H4: Hole, kbd:M2_HOLE_v3, F.Cu at (124.2, 35.7)
- added H5: Hole, kbd:M2_HOLE_v3, F.Cu at (227.3, 33.4)
- added H6: Hole, kbd:M2_HOLE_v3, F.Cu at (199.0, 82.2)
- added H7: Hole, kbd:M2_HOLE_v3, F.Cu at (154.7, 54.8)
- added R7: 1M, Resistor_SMD:R_0805_2012Metric, B.Cu at (222.8, 22.0)
- added U2: SRV05-4, Package_TO_SOT_SMD:SOT-23-6, B.Cu at (229.8, 26.1)
- added USB1: HRO-TYPE-C-31-M-12, Type-C:HRO-TYPE-C-31-M-12, B.Cu at (229.8, 15.2)
- C1: value 22pF -> 4.7n
- R1: moved to B.Cu
- SW1: footprint rainstuff:tht-reset -> random-keyboard-parts:SKQG-1155865; moved to B.Cu
- Y1: value 16MHz -> Resonator_Small; footprint Crystal:Crystal_SMD_3225-4Pin_3.2x2.5mm -> Crystal:Resonator_SMD_muRata_CSTxExxV-3Pin_3.0x1.1mm
- moved SW1 167.3 mm to (20.8, 56.6), turned to 90 degrees
- moved C1 99.8 mm to (222.8, 19.9), turned to 0 degrees
- moved C4 33.0 mm to (173.9, 78.4), turned to 315 degrees
- moved R4 32.1 mm to (161.6, 71.3), turned to 225 degrees
- moved C6 31.3 mm to (166.9, 71.4), turned to 135 degrees
- moved C7 24.6 mm to (169.3, 89.7), turned to 270 degrees
- moved C8 22.6 mm to (155.1, 77.8), turned to 225 degrees
- moved R1 20.2 mm to (166.4, 90.6), turned to 225 degrees
- moved D41 15.9 mm to (146.1, 85.7)
- moved C5 15.2 mm to (160.9, 90.1), turned to 135 degrees
- moved C3 13.5 mm to (171.2, 87.5), turned to 315 degrees
- moved R6 13.3 mm to (236.9, 17.8), turned to 0 degrees
- moved R5 12.2 mm to (222.8, 17.8), turned to 180 degrees
- moved R3 8.92 mm to (230.8, 33.9)
- moved R2 8.89 mm to (232.8, 33.9)
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Connections:
- net Net-(R2-Pad1) renamed DP+
- net Net-(R3-Pad1) renamed DP-
- C4 pad 1: VCC -> +5V
- C5 pad 1: VCC -> +5V
- C6 pad 1: VCC -> +5V
- C7 pad 1: VCC -> +5V
- C8 pad 1: VCC -> +5V
- F1 pad 1: VCC -> +5V
- F1 pad 2: Net-(F1-Pad2) -> VCC
- R1 pad 1: VCC -> +5V
- U1 pad 14: VCC -> +5V
- U1 pad 17: Net-(C1-Pad2) -> Net-(U1-Pad17)
- U1 pad 18: Net-(U1-Pad18) -> D
- U1 pad 19: Net-(U1-Pad19) -> C
- U1 pad 2: VCC -> +5V
- U1 pad 20: Net-(U1-Pad20) -> 6
- U1 pad 21: Net-(U1-Pad21) -> 7
- U1 pad 22: Net-(U1-Pad22) -> 8
- U1 pad 24: VCC -> +5V
- U1 pad 25: Net-(U1-Pad25) -> 0
- U1 pad 26: Net-(U1-Pad26) -> 1
- U1 pad 27: Net-(U1-Pad27) -> 2
- U1 pad 28: Net-(U1-Pad28) -> 3
- U1 pad 29: Net-(U1-Pad29) -> 4
- U1 pad 30: Net-(U1-Pad30) -> 5
- U1 pad 31: Net-(U1-Pad31) -> B
- U1 pad 32: Net-(U1-Pad32) -> A
- U1 pad 34: VCC -> +5V
- U1 pad 36: Net-(U1-Pad36) -> 9
- U1 pad 37: Net-(U1-Pad37) -> 10
- U1 pad 38: Net-(U1-Pad38) -> 11
- U1 pad 44: VCC -> +5V
- U1 pad 7: VCC -> +5V
- Y1 pad 1: Net-(C1-Pad2) -> Net-(U1-Pad17)
Routing:
- net +5V: track 0.00 -> 193.4 mm, vias 0 -> 6
- net Net-(R1-Pad2): track 0.00 -> 165.7 mm, vias 0 -> 2
- net A: track 226.7 -> 376.5 mm, vias 0 -> 4
- net 0: track 60.2 -> 205.2 mm
- net B: track 216.7 -> 358.0 mm, vias 0 -> 4
- net 1: track 68.9 -> 188.7 mm
- net 2: track 65.0 -> 171.7 mm
- net 11: track 40.2 -> 143.7 mm, vias 0 -> 3
- net DP+: track 0.00 -> 100.0 mm
- net DP-: track 0.00 -> 100.0 mm
- net 3: track 44.1 -> 118.1 mm, vias 0 -> 1
- net 10: track 73.3 -> 135.6 mm, vias 0 -> 3
- net 4: track 44.0 -> 99.4 mm, vias 0 -> 1
- net 8: track 44.0 -> 89.4 mm, vias 0 -> 3
- net 9: track 62.1 -> 106.4 mm, vias 0 -> 1
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