File: vanish.sch (KiCad schematic (older format))
At the start: 111 parts, among them J1 USB_C_Receptacle_USB2.0, SW1 SW_Push, U1 ATmega32U4-AU, Y1 16MHz

Commit message: pcb woirk
Parts:
- removed D40, D42: D_Small, Diode_SMD:D_SOD-123, symbol Device:D_Small
- removed MX40, MX41, MX43: MX-NoLED, MX_Alps_Hybrid:MX-2U-ReversedStabilizers-NoLED, symbol MX_Alps_Hybrid:MX-NoLED
- removed MX45: MX-NoLED, MX_Alps_Hybrid:MX-1.25U-NoLED, symbol MX_Alps_Hybrid:MX-NoLED
- added C8: 0.1uF, Capacitor_SMD:C_0805_2012Metric, symbol Device:C_Small
- MX44: footprint MX_Alps_Hybrid:MX-1U-NoLED -> MX_Alps_Hybrid:MX-1.25U-NoLED
- MX47: footprint MX_Alps_Hybrid:MX-1.25U-NoLED -> MX_Alps_Hybrid:MX-1U-NoLED
Changed lines of the file:
@@
-$EndComp
-$Comp
-L Device:D_Small D40
-U 1 1 5FAA4719
-P 3100 3150
-F 0 "D40" V 3146 3082 50  0000 R CNN
-F 1 "D_Small" V 3055 3082 50  0000 R CNN
-F 2 "Diode_SMD:D_SOD-123" V 3100 3150 50  0001 C CNN
-F 3 "~" V 3100 3150 50  0001 C CNN
-	1    3100 3150
-	0    -1   -1   0
-$EndComp
-$Comp
-L MX_Alps_Hybrid:MX-NoLED MX41
-U 1 1 5FAA471F
-P 3650 2900
-F 0 "MX41" H 3683 3123 60  0000 C CNN
-F 1 "MX-NoLED" H 3683 3049 20  0000 C CNN
-F 2 "MX_Alps_Hybrid:MX-2U-ReversedStabilizers-NoLED" H 3025 2875 60  0001 C CNN
-F 3 "" H 3025 2875 60  0001 C CNN
-	1    3650 2900
-	1    0    0    -1
 $EndComp
 $Comp
@@
 $EndComp
 $Comp
-L MX_Alps_Hybrid:MX-NoLED MX43
-U 1 1 5FAA472B
-P 4150 2900
-F 0 "MX43" H 4183 3123 60  0000 C CNN
-F 1 "MX-NoLED" H 4183 3049 20  0000 C CNN
-F 2 "MX_Alps_Hybrid:MX-2U-ReversedStabilizers-NoLED" H 3525 2875 60  0001 C CNN
-F 3 "" H 3525 2875 60  0001 C CNN
-	1    4150 2900
-	1    0    0    -1
-$EndComp
-$Comp
-L Device:D_Small D42
-U 1 1 5FAA4731
-P 4100 3150
-F 0 "D42" V 4146 3082 50  0000 R CNN
-F 1 "D_Small" V 4055 3082 50  0000 R CNN
-F 2 "Diode_SMD:D_SOD-123" V 4100 3150 50  0001 C CNN
-F 3 "~" V 4100 3150 50  0001 C CNN
-	1    4100 3150
-	0    -1   -1   0
-$EndComp
-$Comp
 L MX_Alps_Hybrid:MX-NoLED MX44
 U 1 1 5FAA4737
@@
 F 0 "MX44" H 5433 3123 60  0000 C CNN
 F 1 "MX-NoLED" H 5433 3049 20  0000 C CNN
-F 2 "MX_Alps_Hybrid:MX-1U-NoLED" H 4775 2875 60  0001 C CNN
+F 2 "MX_Alps_Hybrid:MX-1.25U-NoLED" H 4775 2875 60  0001 C CNN
 F 3 "" H 4775 2875 60  0001 C CNN
 	1    5400 2900
@@
 F 0 "MX47" H 6433 3123 60  0000 C CNN
 F 1 "MX-NoLED" H 6433 3049 20  0000 C CNN
-F 2 "MX_Alps_Hybrid:MX-1.25U-NoLED" H 5775 2875 60  0001 C CNN
+F 2 "MX_Alps_Hybrid:MX-1U-NoLED" H 5775 2875 60  0001 C CNN
 F 3 "" H 5775 2875 60  0001 C CNN
 	1    6400 2900
@@
 $EndComp
 $Comp
-L MX_Alps_Hybrid:MX-NoLED MX45
-U 1 1 5FAB49EF
-P 5450 2900
-F 0 "MX45" H 5483 3123 60  0000 C CNN
-F 1 "MX-NoLED" H 5483 3049 20  0000 C CNN
-F 2 "MX_Alps_Hybrid:MX-1.25U-NoLED" H 4825 2875 60  0001 C CNN
-F 3 "" H 4825 2875 60  0001 C CNN
-	1    5450 2900
-	1    0    0    -1
-$EndComp
-$Comp
 L MCU_Microchip_ATmega:ATmega32U4-AU U1
 U 1 1 5FAB6D34
@@
 Wire Wire Line
 	2550 1550 2550 2200
-$Comp
-L MX_Alps_Hybrid:MX-NoLED MX40
-U 1 1 5FAA4713
-P 3150 2900
-F 0 "MX40" H 3183 3123 60  0000 C CNN
-F 1 "MX-NoLED" H 3183 3049 20  0000 C CNN
-F 2 "MX_Alps_Hybrid:MX-2U-ReversedStabilizers-NoLED" H 2525 2875 60  0001 C CNN
-F 3 "" H 2525 2875 60  0001 C CNN
-	1    3150 2900
-	1    0    0    -1
-$EndComp
 Wire Wire Line
 	3300 2850 3300 2350
@@
 Wire Wire Line
 	3850 2850 3800 2850
-Connection ~ 3800 2850
 Wire Wire Line
 	4300 2850 4300 2350
@@
 Wire Wire Line
 	1850 3250 1350 3250
-Connection ~ 3100 3250
-Wire Wire Line
-	3100 3250 1850 3250
 Connection ~ 3600 3250
-Wire Wire Line
-	3600 3250 3100 3250
-Connection ~ 4100 3250
-Wire Wire Line
-	4100 3250 3600 3250
 Connection ~ 5350 3250
-Wire Wire Line
-	5350 3250 4100 3250
 Connection ~ 5850 3250
 Wire Wire Line
@@
 Wire Wire Line
 	3650 3050 3600 3050
-Connection ~ 3600 3050
 $Comp
 L Connector:USB_C_Receptacle_USB2.0 J1
@@
 Wire Wire Line
 	6650 6150 6800 6150
+$Comp
+L Device:C_Small C8
+U 1 1 5FA8A2A3
+P 6600 3850
+F 0 "C8" H 6692 3896 50  0000 L CNN
+F 1 "0.1uF" H 6692 3805 50  0000 L CNN
+F 2 "Capacitor_SMD:C_0805_2012Metric" H 6600 3850 50  0001 C CNN
+F 3 "~" H 6600 3850 50  0001 C CNN
+	1    6600 3850
+	1    0    0    -1
+$EndComp
+Connection ~ 6900 3750
+Wire Wire Line
+	6900 3750 6600 3750
+Wire Wire Line
+	6600 3950 6900 3950
+Connection ~ 6900 3950
+Wire Wire Line
+	1850 3250 3600 3250
+Wire Wire Line
+	3600 3250 5350 3250
 $EndSCHEMATC

Commit message: done
Parts:
- removed C2: 22pF, Capacitor_SMD:C_0805_2012Metric, symbol Device:C_Small
- removed J1: USB_C_Receptacle_USB2.0, Connector_USB:USB_C_Receptacle_GCT_USB4085, symbol Connector:USB_C_Receptacle_USB2.0
- removed Y1: 16MHz, Crystal:Crystal_SMD_3225-4Pin_3.2x2.5mm, symbol Device:Crystal_GND24_Small
- added H1, H2, H3, H4, H5, H6, H7: Hole, kbd:M2_HOLE_v3, symbol keebio:Hole
- added R7: 1M, Resistor_SMD:R_0805_2012Metric, symbol Device:R_Small
- added U2: SRV05-4, Package_TO_SOT_SMD:SOT-23-6, symbol Power_Protection:SRV05-4
- added USB1: HRO-TYPE-C-31-M-12, Type-C:HRO-TYPE-C-31-M-12, symbol Type-C:HRO-TYPE-C-31-M-12
- added Y1: Resonator_Small, Crystal:Resonator_SMD_muRata_CSTxExxV-3Pin_3.0x1.1mm, symbol Device:Resonator_Small
- C1: value 22pF -> 4.7n
- SW1: footprint rainstuff:tht-reset -> random-keyboard-parts:SKQG-1155865
Connections:
- net labels added: +5V, DP+, DP-
- wire segments 153 -> 157
Other:
- moved on the sheet: F1, R2, R3, R5, R6

Commit message: yup
Parts:
- F1: value Polyfuse_Small -> 500mA
Changed lines of the file:
@@
 P 7800 4750
 F 0 "F1" V 7595 4750 50  0000 C CNN
-F 1 "Polyfuse_Small" V 7686 4750 50  0000 C CNN
+F 1 "500mA" V 7686 4750 50  0000 C CNN
 F 2 "Fuse:Fuse_1206_3216Metric" H 7850 4550 50  0001 L CNN
 F 3 "~" H 7800 4750 50  0001 C CNN
